File: loop-sampler/loop-sampler.kicad_sch (KiCad schematic)
At the start: 27 parts, among them J1 3.5mm_Stereo, J2 3.5mm_Stereo, J3 3.5mm_Stereo, J4 3.5mm_Stereo, SW1 SW_SPDT_MSM

Commit message: Implements forward/reverse mode switch on GP16/17
Connections:
- net GPIO19 is gone; now on net ENC_SW: EXT1.9
- net ENC_SW: no longer EXT1.24
- net FM_IN: now also EXT2.29; no longer EXT2.27
- net GPIO43 renamed GPIO42
- net GPIO42: now also EXT2.27; no longer EXT2.29
- new net GPIO8\QMI_CS1n: EXT1.24
Changed lines of the file:
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@@
 	)
 	(label "ENC_SW"
-		(at 128.27 130.81 180)
-		(effects
-			(font
-				(size 1.27 1.27)
-			)
-			(justify right bottom)
+		(at 189.23 113.03 0)
+		(effects
+			(font
+				(size 1.27 1.27)
+			)
+			(justify left bottom)
 		)
 	)
@@
 	)
 	(label "TUNE_KNOB"
-		(at 344.17 138.43 0)
+		(at 344.17 135.89 0)
 		(effects
 			(font
@@
 	)
 	(label "FM_IN"
-		(at 344.17 135.89 0)
-		(effects
-			(font
+		(at 344.17 138.43 0)
+		(effects
+			(font
